Commit message: modified the imu.xacro

File: src/agv_description/urdf/sensors/imu_gazebo.xacro (robot description, xacro)
@@ -14,5 +14,5 @@
                 <origin xyz=" 0 0 0 " rpy="0 0 0" />
                 <geometry>
-                    <box size="0.36 0.36 0.17" />
+                    <box size="0.036 0.036 0.017" />
                 </geometry>
                 <material name="black"/>
@@ -21,5 +21,5 @@
                 <origin xyz="0.0 0.0 0.0" rpy="0 0 0" />
                 <geometry>
-                    <cylinder length="0.06" radius="0.05"/>
+                    <box size="0.036 0.036 0.017" />
                 </geometry>
             </collision>
