Commit message: Update imu.xacro

File: src/agv_description/urdf/sensors/imu.xacro (robot description, xacro)
@@ -6,13 +6,5 @@
                 <origin xyz=" 0 0 0 " rpy="0 0 0" />
                 <geometry>
-<<<<<<< HEAD
-<<<<<<< HEAD
-                    <box size="0.36 0.36 0.17" />
-=======
                     <box size="0.036 0.036 0.017" />
->>>>>>> dev1109
-=======
-                    <box size="0.036 0.036 0.017" />
->>>>>>> upstream/develop
                 </geometry>
                 <material name="black"/>
