Commit message: add imu.xacro in agv_description

File: src/agv_description/urdf/agv_with_sensors.xacro (robot description, xacro)
@@ -3,9 +3,10 @@
     <xacro:include filename="$(find agv_description)/urdf/agv_base.xacro" />
     <xacro:include filename="$(find agv_description)/urdf/sensors/lidar.xacro" />
+    <xacro:include filename="$(find agv_description)/urdf/sensors/imu.xacro" />
+    <agv_base/>
+    <!-- Lidar -->
     <xacro:property name="lidar_offset_x" value="0.40" />
     <xacro:property name="lidar_offset_y" value="0" />
     <xacro:property name="lidar_offset_z" value="0.185" />
-    <agv_base/>
-    <!-- Lidar -->
     <joint name="laser_joint" type="fixed">
         <origin xyz="${lidar_offset_x} ${lidar_offset_y} ${lidar_offset_z}" rpy="0 0 0" />
@@ -14,3 +15,13 @@
     </joint>
     <xacro:lidar prefix="laser"/>
+    <!-- imu -->
+    <xacro:property name="imu_offset_x" value="-0.28" />
+    <xacro:property name="imu_offset_y" value="-0.07" />
+    <xacro:property name="imu_offset_z" value="0.01" />
+    <joint name="imu_joint" type="fixed">
+        <origin xyz="${imu_offset_x} ${imu_offset_y} ${imu_offset_z}" rpy="0 0 0"/>
+        <parent link="base_link"/>
+        <child link="imu_link"/>
+    </joint>
+    <xacro::imu prefix="imu"/>
 </robot>

Commit message: modified the imu.xacro

File: src/agv_description/urdf/agv_with_sensors.xacro (robot description, xacro)
@@ -24,4 +24,4 @@
         <child link="imu_link"/>
     </joint>
-    <xacro::imu prefix="imu"/>
+    <xacro:imu prefix="imu"/>
 </robot>

File: src/agv_description/urdf/sensors/imu.xacro (robot description, xacro)
@@ -6,5 +6,5 @@
                 <origin xyz=" 0 0 0 " rpy="0 0 0" />
                 <geometry>
-                    <box size="0.36 0.36 0.17" />
+                    <box size="0.036 0.036 0.017" />
                 </geometry>
                 <material name="black"/>

File: src/agv_description/urdf/sensors/lidar_gazebo.xacro (robot description, xacro)
@@ -12,5 +12,5 @@
             </inertial>
             <visual>
-		<origin xyz=" 0 0 0 " rpy="0 0 0" />
+		        <origin xyz=" 0 0 0 " rpy="0 0 0" />
                 <geometry>
                     <cylinder length="0.05" radius="0.05"/>

Commit message: modified agv_run.launch,main.cpp,drivertest_node.cpp

File: src/agv_description/urdf/agv_with_sensors.xacro (robot description, xacro)
@@ -2,10 +2,11 @@
 <robot name="agv" xmlns:xacro="http://www.ros.org/wiki/xacro">
     <xacro:include filename="$(find agv_description)/urdf/agv_base.xacro" />
-    <xacro:include filename="$(find agv_description)/urdf/lidar.xacro" />
+    <xacro:include filename="$(find agv_description)/urdf/sensors/lidar.xacro" />
+    <xacro:include filename="$(find agv_description)/urdf/sensors/imu.xacro" />
+    <agv_base/>
+    <!-- Lidar -->
     <xacro:property name="lidar_offset_x" value="0.40" />
     <xacro:property name="lidar_offset_y" value="0" />
     <xacro:property name="lidar_offset_z" value="0.185" />
-    <agv_base/>
-    <!-- Lidar -->
     <joint name="laser_joint" type="fixed">
         <origin xyz="${lidar_offset_x} ${lidar_offset_y} ${lidar_offset_z}" rpy="0 0 0" />
@@ -14,3 +15,13 @@
     </joint>
     <xacro:lidar prefix="laser"/>
+    <!-- imu -->
+    <xacro:property name="imu_offset_x" value="-0.28" />
+    <xacro:property name="imu_offset_y" value="-0.07" />
+    <xacro:property name="imu_offset_z" value="0.01" />
+    <joint name="imu_joint" type="fixed">
+        <origin xyz="${imu_offset_x} ${imu_offset_y} ${imu_offset_z}" rpy="0 0 0"/>
+        <parent link="base_link"/>
+        <child link="imu_link"/>
+    </joint>
+    <xacro:imu prefix="imu"/>
 </robot>
